File: kicad/fan_controller.kicad_pcb (KiCad board)
At the start: 2 copper layers, 60 x 37 mm, 62 parts, among them P1 CONN_01X04, P2 CONN_01X05, P3 CONN_01X04, P4 CONN_01X04, P5 CONN_01X04, P6 CONN_01X04, Q1 Q_NPN_BEC, Q2 Q_NPN_BEC, Q3 Q_NPN_BEC, Q4 Q_NPN_BEC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

Commit message: Added LEDs, fixed #2
Parts:
- removed G***: LOGO, lib_pcb:for_embed_logo
- removed the REF** at (161.0, 82.9)
- removed the REF** at (117.0, 61.9)
- removed W1, W2, W3, W4: TEST_1P, Connect:PINTST
- added D1: LED, Diodes_SMD:D_0805, B.Cu at (155.8, 65.7)
- added D2: LED, Diodes_SMD:D_0805, B.Cu at (147.8, 65.7)
- added D3: LED, Diodes_SMD:D_0805, B.Cu at (139.8, 65.7)
- added D4: LED, Diodes_SMD:D_0805, B.Cu at (131.8, 65.7)
- added R19: 1.0k, Resistors_SMD:R_0603, B.Cu at (131.8, 62.3)
- added R5: 1k, Diodes_SMD:D_0805, B.Cu at (136.4, 87.7)
- added R6: 1.0k, Resistors_SMD:R_0603, B.Cu at (139.8, 87.7)
- added R7: 1.0k, Resistors_SMD:R_0603, B.Cu at (155.8, 62.3)
- added R8: 1.0k, Resistors_SMD:R_0603, B.Cu at (147.8, 62.3)
- added R9: 1.0k, Resistors_SMD:R_0603, B.Cu at (139.8, 62.3)
- R1, R10, R11, R12, R13, R3, R4: footprint kicad_pcb:SM_0603 -> Resistors_SMD:R_0603
- R14, R15, R16, R17, R18, R2: value 1k -> 1.0k; footprint kicad_pcb:SM_0603 -> Resistors_SMD:R_0603
- moved C7 2.52 mm to (159.6, 65.5)
Connections:
- net Net-(P1-Pad3) renamed /sense_out
- U1 pad 16: (no net) -> Net-(U1-Pad16)
- U1 pad 22: (no net) -> Net-(U1-Pad22)
- U1 pad 26: (no net) -> Net-(U1-Pad26)
Routing:
- net /pwm0(OC2B): track 17.2 -> 26.5 mm, vias 0 -> 2
- net /pwm1(OC5): track 13.8 -> 22.8 mm, vias 0 -> 2
- net /pwm3(OC1E): track 17.5 -> 25.9 mm, vias 0 -> 2
- net /pwm2(OC4): track 7.77 -> 13.0 mm
- net /sense1: track 19.8 -> 24.8 mm
- net Net-(U1-Pad9): track 4.59 -> 0.00 mm
- net Net-(U1-Pad12): track 4.46 -> 0.00 mm
- net Net-(U1-Pad11): track 3.90 -> 0.00 mm
- net +5V: track 66.9 -> 69.9 mm
- net GND: track 35.8 -> 38.4 mm
- net /sense0(CN13): track 25.9 -> 28.5 mm
- net Net-(D4-Pad1): track 0.00 -> 1.60 mm
- net Net-(D3-Pad1): track 0.00 -> 1.60 mm
- net Net-(D2-Pad1): track 0.00 -> 1.60 mm
- net Net-(D1-Pad1): track 0.00 -> 1.60 mm
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Other:
- board text added: "for(embed) www.forembed.com fan controller, v1.2"
- board text removed: "for(embed) www.forembed.com fan controller, v1.1"

Commit message: Added logo
Parts:
- added G***: LOGO, footprints:logo-forembed, F.Cu at (129.3, 79.8)
Changed lines of the file:
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@@
     (tracks 311)
     (zones 0)
-    (modules 65)
+    (modules 66)
     (nets 44)
   )
@@
     )
   )
+  (module footprints:logo-forembed (layer F.Cu)
+    (at 129.266 79.832)
+    (fp_text reference G*** (at 0 0) (layer F.SilkS) hide
+      (effects (font (thickness 0.3)))
+    )
+    (fp_text value LOGO (at 0.75 0) (layer F.SilkS) hide
+      (effects (font (thickness 0.3)))
+    )
+    (fp_poly (pts (xy 0.125042 -3.997651) (xy 0.228182 -3.939989) (xy 0.286285 -3.85872) (xy 0.302344 -3.787111)
+      (xy 0.315169 -3.658717) (xy 0.323623 -3.489295) (xy 0.326572 -3.300292) (xy 0.326572 -2.830285)
+      (xy 0.689429 -2.830285) (xy 0.689429 -3.282149) (xy 0.692754 -3.474934) (xy 0.701924 -3.640967)
+      (xy 0.715727 -3.764252) (xy 0.730422 -3.823983) (xy 0.808538 -3.921577) (xy 0.916191 -3.967347)
+      (xy 1.032185 -3.961366) (xy 1.135325 -3.903703) (xy 1.193428 -3.822434) (xy 1.209518 -3.751061)
+      (xy 1.222426 -3.623896) (xy 1.230903 -3.457691) (xy 1.233715 -3.282149) (xy 1.233715 -2.830285)
+      (xy 2.830286 -2.830285) (xy 2.830286 -1.197428) (xy 3.318436 -1.197428) (xy 3.524858 -1.1943)
+      (xy 3.699711 -1.185573) (xy 3.82905 -1.172237) (xy 3.896555 -1.156436) (xy 3.994149 -1.078319)
+      (xy 4.039919 -0.970666) (xy 4.033938 -0.854672) (xy 3.976275 -0.751532) (xy 3.895006 -0.69343)
+      (xy 3.823208 -0.677409) (xy 3.693688 -0.664665) (xy 3.521257 -0.656231) (xy 3.320732 -0.653143)
+      (xy 3.318436 -0.653142) (xy 2.830286 -0.653143) (xy 2.830286 -0.254) (xy 3.300293 -0.254)
+      (xy 3.499958 -0.250775) (xy 3.670413 -0.241831) (xy 3.796717 -0.22826) (xy 3.860269 -0.213007)
+      (xy 3.957863 -0.13489) (xy 4.003634 -0.027238) (xy 3.997652 0.088756) (xy 3.939989 0.191897)
+      (xy 3.85872 0.249999) (xy 3.787111 0.266059) (xy 3.658718 0.278884) (xy 3.489295 0.287337)
+      (xy 3.300293 0.290286) (xy 2.830286 0.290286) (xy 2.830286 0.689429) (xy 3.318436 0.689429)
+      (xy 3.524858 0.692557) (xy 3.699711 0.701284) (xy 3.82905 0.71462) (xy 3.896555 0.730422)
+      (xy 3.994149 0.808538) (xy 4.039919 0.916191) (xy 4.033938 1.032185) (xy 3.976275 1.135325)
+      (xy 3.895006 1.193428) (xy 3.823208 1.209448) (xy 3.693688 1.222193) (xy 3.521257 1.230626)
+      (xy 3.320732 1.233714) (xy 3.318436 1.233715) (xy 2.830286 1.233715) (xy 2.830286 2.830286)
+      (xy 1.233715 2.830286) (xy 1.233715 3.318436) (xy 1.230586 3.524858) (xy 1.22186 3.699711)
+      (xy 1.208524 3.82905) (xy 1.192722 3.896555) (xy 1.114605 3.994149) (xy 1.006953 4.039919)
+      (xy 0.890959 4.033938) (xy 0.787818 3.976275) (xy 0.729716 3.895006) (xy 0.713696 3.823208)
+      (xy 0.700951 3.693688) (xy 0.692517 3.521257) (xy 0.689429 3.320732) (xy 0.689429 2.830286)
+      (xy 0.326572 2.830286) (xy 0.326572 3.300293) (xy 0.323347 3.499958) (xy 0.314403 3.670413)
+      (xy 0.300833 3.796717) (xy 0.285579 3.860269) (xy 0.207463 3.957863) (xy 0.09981 4.003634)
+      (xy -0.016184 3.997652) (xy -0.119324 3.939989) (xy -0.177427 3.85872) (xy -0.193486 3.787111)
+      (xy -0.206311 3.658718) (xy -0.214765 3.489295) (xy -0.217714 3.300293) (xy -0.217714 2.830286)
+      (xy -0.653143 2.830286) (xy -0.653143 3.318436) (xy -0.656054 3.554656) (xy -0.666524 3.729331)
+      (xy -0.687152 3.853318) (xy -0.720542 3.937475) (xy -0.769294 3.992659) (xy -0.822137 4.023713)
+      (xy -0.90332 4.055487) (xy -0.963523 4.053737) (xy -1.039074 4.021561) (xy -1.09874 3.980624)
+      (xy -1.141869 3.917252) (xy -1.170868 3.820759) (xy -1.188145 3.680458) (xy -1.196107 3.485661)
+      (xy -1.197428 3.318436) (xy -1.197428 2.830286) (xy -2.830285 2.830286) (xy -2.830285 1.233715)
+      (xy -1.850571 1.233715) (xy -1.850571 1.886857) (xy -1.197428 1.886857) (xy -1.197428 1.233715)
+      (xy -0.653143 1.233715) (xy -0.653143 1.886857) (xy -0.217714 1.886857) (xy -0.217714 1.233715)
+      (xy 0.326572 1.233715) (xy 0.326572 1.886857) (xy 0.689429 1.886857) (xy 0.689429 1.233715)
+      (xy 1.233715 1.233715) (xy 1.233715 1.886857) (xy 1.886857 1.886857) (xy 1.886857 1.233715)
+      (xy 1.233715 1.233715) (xy 0.689429 1.233715) (xy 0.326572 1.233715) (xy -0.217714 1.233715)
+      (xy -0.653143 1.233715) (xy -1.197428 1.233715) (xy -1.850571 1.233715) (xy -2.830285 1.233715)
+      (xy -3.264007 1.233715) (xy -3.449783 1.230283) (xy -3.611367 1.220882) (xy -3.731651 1.20685)
+      (xy -3.787697 1.192722) (xy -3.885291 1.114605) (xy -3.931062 1.006953) (xy -3.92508 0.890959)
+      (xy -3.867417 0.787818) (xy -3.786148 0.729716) (xy -3.715067 0.713605) (xy -3.589241 0.700611)
+      (xy -3.426476 0.692107) (xy -3.264007 0.689429) (xy -2.830285 0.689429) (xy -2.830285 0.290286)
+      (xy -1.850571 0.290286) (xy -1.850571 0.689429) (xy -1.197428 0.689429) (xy -1.197428 0.290286)
+      (xy -0.653143 0.290286) (xy -0.653143 0.689429) (xy -0.217714 0.689429) (xy -0.217714 0.290286)
+      (xy 0.326572 0.290286) (xy 0.326572 0.689429) (xy 0.689429 0.689429) (xy 0.689429 0.290286)
+      (xy 1.233715 0.290286) (xy 1.233715 0.689429) (xy 1.886857 0.689429) (xy 1.886857 0.290286)
+      (xy 1.233715 0.290286) (xy 0.689429 0.290286) (xy 0.326572 0.290286) (xy -0.217714 0.290286)
+      (xy -0.653143 0.290286) (xy -1.197428 0.290286) (xy -1.850571 0.290286) (xy -2.830285 0.290286)
+      (xy -3.282149 0.290286) (xy -3.474934 0.286961) (xy -3.640967 0.277791) (xy -3.764252 0.263988)
+      (xy -3.823983 0.249293) (xy -3.921577 0.171177) (xy -3.967347 0.063524) (xy -3.961366 -0.05247)
+      (xy -3.903703 -0.15561) (xy -3.822434 -0.213713) (xy -3.751061 -0.229803) (xy -3.623896 -0.242711)
+      (xy -3.457691 -0.251188) (xy -3.282149 -0.254) (xy -2.830285 -0.254) (xy -2.830285 -0.653143)
+      (xy -1.850571 -0.653143) (xy -1.850571 -0.254) (xy -1.197428 -0.254) (xy -1.197428 -0.653143)
+      (xy -0.653143 -0.653143) (xy -0.653143 -0.254) (xy -0.217714 -0.254) (xy -0.217714 -0.653143)
+      (xy 0.326572 -0.653143) (xy 0.326572 -0.254) (xy 0.689429 -0.254) (xy 0.689429 -0.653143)
+      (xy 1.233715 -0.653143) (xy 1.233715 -0.254) (xy 1.886857 -0.254) (xy 1.886857 -0.653143)
+      (xy 1.233715 -0.653143) (xy 0.689429 -0.653143) (xy 0.326572 -0.653143) (xy -0.217714 -0.653143)
+      (xy -0.653143 -0.653143) (xy -1.197428 -0.653143) (xy -1.850571 -0.653143) (xy -2.830285 -0.653143)
+      (xy -3.264007 -0.653142) (xy -3.449783 -0.656574) (xy -3.611367 -0.665975) (xy -3.731651 -0.680008)
+      (xy -3.787697 -0.694135) (xy -3.885291 -0.772252) (xy -3.931062 -0.879904) (xy -3.92508 -0.995898)
+      (xy -3.867417 -1.099039) (xy -3.786148 -1.157141) (xy -3.715067 -1.173252) (xy -3.589241 -1.186246)
+      (xy -3.426476 -1.19475) (xy -3.264007 -1.197428) (xy -2.830285 -1.197428) (xy -1.850571 -1.197428)
+      (xy -1.197428 -1.197428) (xy -1.197428 -1.542143) (xy -1.198144 -1.701857) (xy -1.202573 -1.80259)
+      (xy -1.214139 -1.857929) (xy -1.236267 -1.881463) (xy -1.272379 -1.886781) (xy -1.284281 -1.886857)
+      (xy -0.653143 -1.886857) (xy -0.653143 -1.197428) (xy -0.217714 -1.197428) (xy -0.217714 -1.886857)
+      (xy 0.326572 -1.886857) (xy 0.326572 -1.197428) (xy 0.689429 -1.197428) (xy 0.689429 -1.886857)
+      (xy 1.233715 -1.886857) (xy 1.233715 -1.197428) (xy 1.886857 -1.197428) (xy 1.886857 -1.886857)
+      (xy 1.233715 -1.886857) (xy 0.689429 -1.886857) (xy 0.326572 -1.886857) (xy -0.217714 -1.886857)
+      (xy -0.653143 -1.886857) (xy -1.284281 -1.886857) (xy -1.359001 -1.859368) (xy -1.459931 -1.78702)
+      (xy -1.572513 -1.68499) (xy -1.682186 -1.568455) (xy -1.774392 -1.452592) (xy -1.83457 -1.352579)
+      (xy -1.849926 -1.297214) (xy -1.850571 -1.197428) (xy -2.830285 -1.197428) (xy -2.830285 -1.908585)
+      (xy -1.898763 -2.830285) (xy -1.197428 -2.830285) (xy -1.197428 -3.282149) (xy -1.194213 -3.469674)
+      (xy -1.185401 -3.633793) (xy -1.172242 -3.757754) (xy -1.157141 -3.822434) (xy -1.078889 -3.920551)
+      (xy -0.971172 -3.967042) (xy -0.855186 -3.961836) (xy -0.752125 -3.904863) (xy -0.694135 -3.823983)
+      (xy -0.677308 -3.750396) (xy -0.664071 -3.620271) (xy -0.655635 -3.449603) (xy -0.653143 -3.282149)
+      (xy -0.653143 -2.830285) (xy -0.217714 -2.830285) (xy -0.217714 -3.300292) (xy -0.214489 -3.499957)
+      (xy -0.205545 -3.670412) (xy -0.191975 -3.796716) (xy -0.176721 -3.860268) (xy -0.098605 -3.957862)
+      (xy 0.009048 -4.003633) (xy 0.125042 -3.997651)) (layer F.SilkS) (width 0.01))
+  )
   (dimension 37 (width 0.3) (layer Dwgs.User)
     (gr_text "37.000 mm" (at 99.616 72.432 90) (layer Dwgs.User)
@@
     (effects (font (size 1 1) (thickness 0.25)) (justify mirror))
   )
-  (gr_text "for(embed)\nwww.forembed.com\nfan controller, v1.2" (at 134.766 77.832) (layer F.SilkS)
+  (gr_text "for(embed)\nwww.forembed.com\nfan controller, v1.2" (at 134.666 79.932) (layer F.SilkS)
     (effects (font (size 1.5 1.5) (thickness 0.3)) (justify left))
   )
